File: Spartan2Bone.brd (EAGLE design)
At the start: 100 x 80 mm, 28 parts, among them IC01 XC2S30-5VQG100C100-VQFP-M, IC02 XCF01SVOG20C20-TSSOP-M, IC03 LM2937ET-3.3/NOPB

Commit message: Testing.
Parts:
- moved POWER 87.8 mm to (91.4, 15.7), turned to 90 degrees
- moved MODE0 83.2 mm to (8.91, 32.3), turned to 270 degrees
- moved MODE1 83.2 mm to (8.91, 27.2), turned to 270 degrees
- moved MODE2 83.2 mm to (8.91, 22.1), turned to 270 degrees
- moved PCONF 75.7 mm to (81.9, 15.7), turned to 90 degrees
- moved R1 65.0 mm to (18.5, 32.5)
- moved R2 65.0 mm to (18.5, 27.4)
- moved R3 65.0 mm to (18.5, 22.3)
- moved IC03 53.7 mm to (70.9, 15.1), turned to 90 degrees
- moved C1 32.5 mm to (87.4, 34.7), turned to 180 degrees
- moved IC02 22.0 mm to (78.3, 32.2)
- moved R4 16.8 mm to (50.2, 27.2)
- moved C8 13.3 mm to (32.1, 16.3), turned to 0 degrees
- moved C9 12.8 mm to (32.1, 9.38), turned to 0 degrees
- moved C6 10.1 mm to (43.1, 16.4), turned to 180 degrees
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Connections:
- net DONE: now also R4.2; no longer R4.1
- net GND: now also C2.2, C8.1, C9.1; no longer C2.1, C8.2, C9.2
- net VCCINT: now also C9.2, R4.1; no longer C9.1, R4.2
- net VCCO: now also C2.1, C8.2; no longer C2.2, C8.1
Routing:
- net GND: track 508.1 -> 18.8 mm
- net VCCO: track 321.8 -> 165.6 mm, vias 0 -> 3
- net VCCINT: track 264.9 -> 326.7 mm, vias 0 -> 6
- net DONE: track 8.64 -> 0.00 mm
- net M2: track 5.08 -> 0.00 mm
- net M1: track 5.08 -> 0.00 mm
- net M0: track 5.08 -> 0.00 mm
- net REG33: track 11.8 -> 11.3 mm
- added copper zone on layer 1, net GND
- added copper zone on layer 16, net GND

Commit message: Testing.
Parts:
- moved JTAG 83.2 mm to (91.6, 53.1), turned to 90 degrees
- moved IC02 3.41 mm to (80.2, 35.0)
- moved C1 1.53 mm to (88.8, 35.4), turned to 90 degrees
- moved R3 1.19 mm to (17.3, 22.1)
- moved R1 1.19 mm to (17.3, 32.3)
- moved R2 1.19 mm to (17.3, 27.2)
Routing:
- net VCCINT: track 326.7 -> 335.1 mm
- net GND: track 18.8 -> 24.7 mm

Commit message: Testing.
Parts:
- moved C11 5.43 mm to (70.8, 46.4), turned to 180 degrees
- moved C3 5.12 mm to (70.9, 40.9), turned to 0 degrees
- moved C4 3.18 mm to (34.0, 36.3)
- moved C5 3.17 mm to (41.5, 27.4)
- moved CN2 2.29 mm to (72.6, 70.0)
- moved R1 1.91 mm to (17.3, 30.4)
- moved C1 1.91 mm to (88.8, 33.5)
- moved C10 1.91 mm to (59.4, 55.1)
- moved C12 1.91 mm to (33.9, 46.6)
- moved C13 1.91 mm to (41.4, 55.1)
- moved C7 1.91 mm to (43.2, 7.53)
- moved CN1 1.91 mm to (31.1, 70.0)
- moved IC01 1.91 mm to (50.1, 41.8)
- moved IC02 1.91 mm to (80.2, 33.1)
- moved IC03 1.91 mm to (70.9, 13.2)
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Routing:
- net VCCINT: track 335.1 -> 0.00 mm, vias 6 -> 0
- net VCCO: track 165.6 -> 0.00 mm, vias 3 -> 0
- net GND: track 24.7 -> 0.00 mm
- net REG33: track 11.3 -> 0.00 mm
- removed copper zone on layer 16, net GND

Commit message: Testing.
Parts:
- moved C4 32.8 mm to (60.9, 55.1), turned to 180 degrees
- moved C10 32.0 mm to (32.4, 38.0), turned to 270 degrees
- moved C2 9.95 mm to (51.2, 24.4), turned to 180 degrees
- moved R4 5.25 mm to (53.8, 21.5)
- moved IC02 3.56 mm to (76.9, 31.7)
- moved C5 3.23 mm to (42.6, 24.4), turned to 180 degrees
- moved C1 1.56 mm to (89.0, 31.9), turned to 0 degrees
- moved C12 1.54 mm to (32.4, 46.5)
- moved C11 0.10 mm to (70.9, 46.5)
- turned C3 to 180 degrees
Connections:
- net GND: now also C3.1; no longer C3.2
- net VCCINT: now also C3.2; no longer C3.1
Routing:
- net GND: track 0.00 -> 437.1 mm, vias 0 -> 6
- net VCCO: track 0.00 -> 376.2 mm, vias 0 -> 9
- net VCCINT: track 0.00 -> 308.6 mm, vias 0 -> 5
- net REG33: track 0.00 -> 11.3 mm
- removed copper zone on layer 1, net GND

Commit message: First completion.
Routing:
- net TCK: track 0.00 -> 119.2 mm, vias 0 -> 2
- net IO18: track 0.00 -> 97.6 mm, vias 0 -> 3
- net TMS: track 0.00 -> 91.4 mm, vias 0 -> 5
- net IO8: track 0.00 -> 90.0 mm, vias 0 -> 2
- net IO17: track 0.00 -> 88.0 mm, vias 0 -> 2
- net IO20: track 0.00 -> 79.7 mm, vias 0 -> 2
- net IO15: track 0.00 -> 71.3 mm, vias 0 -> 4
- net TRDY: track 0.00 -> 61.4 mm, vias 0 -> 2
- net IO16: track 0.00 -> 61.2 mm, vias 0 -> 2
- net IO19: track 0.00 -> 60.4 mm, vias 0 -> 5
- net IRDY: track 0.00 -> 60.0 mm, vias 0 -> 2
- net IO13: track 0.00 -> 59.4 mm, vias 0 -> 3
- net D4: track 0.00 -> 59.1 mm, vias 0 -> 2
- net INIT: track 0.00 -> 58.4 mm, vias 0 -> 3
- net IO21: track 0.00 -> 57.5 mm, vias 0 -> 2
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