File: Spartan2Bone.brd (EAGLE design)
At the start: 100 x 80 mm, 28 parts, among them IC01 XC2S30-5VQG100C100-VQFP-M, IC02 XCF01SVOG20C20-TSSOP-M, IC03 LM2937ET-3.3/NOPB

Commit message: Fixed board design.
Parts:
- removed MODE0, MODE1, MODE2: (no value), jumper:JP1
- removed POWER: (no value), jumper:JP2
- added CN4: POWER, jumper:JP2
- added JP1: MODE0, jumper:JP1
- added JP2: MODE1, jumper:JP1
- added JP3: MODE2, jumper:JP1
- CN1: value (none) -> IO[1..28]
- CN2: value (none) -> GCK RDY CNT D[0..7]
- CN3: value (none) -> JTAG
- CN5: value (none) -> PCONF
- moved C1 21.3 mm to (70.2, 21.8), turned to 270 degrees
- moved IC03 0.56 mm to (71.3, 12.7)
- turned C10 to 90 degrees
- turned C11 to 0 degrees
- turned C3 to 0 degrees
- turned C4 to 0 degrees
- turned C5 to 0 degrees
- turned C8 to 180 degrees
- turned C9 to 180 degrees
- turned IC02 to 180 degrees
- renumbered JTAG to CN3, PCONF to CN5
Connections:
- net GND: now also C1.2, C10.2, C11.2, C3.2, C4.2, C5.2, C8.2, C9.2, CN4.3; no longer C1.1, C10.1, C11.1, C3.1, C4.1, C5.1, C8.1, C9.1, POWER.3
- net M0: now also JP1.2; no longer MODE0.2
- net M1: now also JP2.2; no longer MODE1.2
- net M2: now also JP3.2; no longer MODE2.2
- net TCK: now also CN3.3; no longer CN3.4
- net TDI: now also CN3.5; no longer CN3.2
- net TDO: now also CN3.4; no longer CN3.5
- net TMS: now also CN3.2; no longer CN3.3
- net VCCINT: now also C1.1, C10.1, C3.1, C5.1, C9.1, CN4.1, JP1.1, JP2.1, JP3.1; no longer C1.2, C10.2, C3.2, C5.2, C9.2, MODE0.1, MODE1.1, MODE2.1, POWER.1
- net VCCO: now also C11.1, C4.1, C8.1, CN4.2; no longer C11.2, C4.2, C8.2, POWER.2
Routing:
- net IO19: track 0.00 -> 141.7 mm, vias 0 -> 2
- net IO15: track 0.00 -> 111.2 mm, vias 0 -> 2
- net IO17: track 0.00 -> 104.1 mm
- net IO18: track 0.00 -> 104.0 mm, vias 0 -> 6
- net TCK: track 0.00 -> 96.4 mm, vias 0 -> 2
- net TMS: track 0.00 -> 95.5 mm, vias 0 -> 4
- net TRDY: track 0.00 -> 95.0 mm, vias 0 -> 1
- net IO16: track 0.00 -> 87.2 mm, vias 0 -> 4
- net IO21: track 0.00 -> 80.8 mm, vias 0 -> 2
- net D6: track 0.00 -> 78.7 mm, vias 0 -> 2
- net IRDY2: track 0.00 -> 76.4 mm, vias 0 -> 1
- net IO14: track 0.00 -> 74.8 mm
- net IO20: track 0.00 -> 70.4 mm, vias 0 -> 4
- net D5: track 0.00 -> 70.3 mm, vias 0 -> 4
- net IO8: track 0.00 -> 69.8 mm, vias 0 -> 2
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- added copper zone on layer 1, net GND
Other:
- board text added: "3.3V"
- board text added: "CNTL"
- board text added: "D[0..7]"
- board text added: "GCLK[0..3]"
- board text added: "GEN3.3V"
- board text added: "GND"
- board text added: "IO[1..8]"
- board text added: "IO[17..24]"
- board text added: "IO[25..28]"
- board text added: "IO[9..16]"
- board text added: "IRDY1,2"
- board text added: "Spartan2Bone 1.0 CC BY-NC-SA"
- board text added: "TCK"
- board text added: "TDI"
- board text added: "TDO"
- board text added: "TMS"
- board text added: "TRDY1,2"
- board text added: "VCCO"
- board text added: "VCOM"
- board text added: "[3.3V]"
- board text added: "https://github.com/kekyo/Spartan2Bone"
